File: dop-module-dc-stepdown-xl4005.kicad_pcb (KiCad board)
At the start: 2 copper layers, 13 parts, among them J101 Conn_01x02, J102 Conn_01x02, U101 XL4005

Commit message: compact layout in progress
Parts:
- added F102: 1A, Fuse:Fuse_1206_3216Metric_Pad1.42x1.75mm_HandSolder, F.Cu at (103.5, 135.3)
- added F103: 1A, Fuse:Fuse_1206_3216Metric_Pad1.42x1.75mm_HandSolder, F.Cu at (101.0, 135.3)
- added F104: 1A, Fuse:Fuse_1206_3216Metric_Pad1.42x1.75mm_HandSolder, F.Cu at (98.4, 135.3)
- F101: value 2A -> 1A
- moved J102 115.2 mm to (138.4, 127.0), turned to 180 degrees
- moved L101 111.1 mm to (130.4, 132.7), turned to 90 degrees
- moved D101 98.2 mm to (120.8, 132.9)
- moved C104 97.1 mm to (129.5, 123.8), turned to 90 degrees
- moved RV101 89.8 mm to (113.7, 135.8), turned to 0 degrees
- moved F101 83.8 mm to (106.0, 135.3), turned to 90 degrees
- moved C101 82.2 mm to (109.3, 135.7), turned to 90 degrees
- moved R101 82.1 mm to (110.9, 131.2), turned to 180 degrees
- moved R102 78.2 mm to (110.9, 128.1), turned to 0 degrees
- moved C102 75.3 mm to (116.2, 123.8), turned to 90 degrees
- moved U101 64.1 mm to (102.2, 124.1), turned to 270 degrees
- moved C103 45.8 mm to (95.9, 116.2), turned to 90 degrees
- moved J101 44.0 mm to (91.4, 127.0), turned to 180 degrees
Connections:
- D101 pad 1: Net-(D101-Pad1) -> GND
- D101 pad 2: GND -> Net-(D101-Pad2)
- D101 pad 3: (no net) -> GND
- F101 pad 1: Net-(D101-Pad1) -> Net-(D101-Pad2)
- L101 pad 1: Net-(D101-Pad1) -> Net-(D101-Pad2)
Routing:
- net Net-(D101-Pad2): track 0.00 -> 50.5 mm, vias 0 -> 20
- net Net-(F101-Pad2): track 0.00 -> 38.6 mm
- net GND: track 0.00 -> 30.0 mm, vias 0 -> 5
- net +5V: track 0.00 -> 27.3 mm
- net Net-(C101-Pad2): track 0.00 -> 20.1 mm
- net +15V: track 0.00 -> 11.8 mm, vias 0 -> 6
- net Net-(R101-Pad1): track 0.00 -> 3.13 mm
- added copper zone on F.Cu, net (none)
- added copper zone on In2.Cu, net (none)
- added copper zone on In2.Cu, net +15V
- added copper zone on In2.Cu, net +5V
- added copper zone on In1.Cu, net GND
- added copper zone on F.Cu, net Net-(D101-Pad2)
- added copper zone on In2.Cu, net Net-(D101-Pad2)
Other:
- copper layers 2 -> 4
- net class 1A added: clearance 0.508, trace_width 0.508, via_dia 0.508, via_drill 0.2032
- net class signal added: clearance 0.2032, trace_width 0.1016, via_dia 0.4064, via_drill 0.2032
- rule trace_min: 0.127 -> 0.1016

Commit message: done : components, traces, pours, edge
Parts:
- moved J102 1.27 mm to (137.2, 127.0)
- moved C103 0.51 mm to (95.4, 116.2)
Routing:
- net GND: track 30.0 -> 69.7 mm, vias 5 -> 33
- net Net-(D101-Pad2): track 50.5 -> 72.5 mm, vias 20 -> 26
- net +5V: track 27.3 -> 48.3 mm
- net +15V: track 11.8 -> 21.5 mm, vias 6 -> 0
- net Net-(F101-Pad2): vias 0 -> 30
- added copper zone on F.Cu, net +15V
- added copper zone on F.Cu, net +5V
- added copper zone on F.Cu, net GND
- added copper zone on In2.Cu, net GND
- added copper zone on B.Cu, net Net-(F101-Pad2)
- removed copper zone on F.Cu, net (none)
- removed copper zone on In2.Cu, net (none)
Other:
- board outline added: 48.3 x 27.9 mm

Commit message: done : silk screen front and back
Parts:
- moved L101 0.63 mm to (129.8, 132.7)
Routing:
- net +5V: track 48.3 -> 85.3 mm, vias 0 -> 10
- net Net-(D101-Pad2): track 72.5 -> 85.1 mm
- net +15V: track 21.5 -> 19.7 mm
Other:
- board text added: "15W should be OK 30W may be OK 45W is too much"
- board text added: "5V 12V"
- board text added: "CC-0 DC stepdown xl4005 module"
- board text added: "GND VIN"
- board text added: "GND VOUT"
- board text added: "WITHOUT WARRANTY of any kind !"

Commit message: done : no more castellation, final
Parts:
- moved C103 0.89 mm to (95.4, 117.1)
- moved C104 0.51 mm to (129.0, 123.8)
- moved C102 0.38 mm to (115.8, 123.8)
Routing:
- net GND: track 69.7 -> 91.5 mm
- net +5V: track 85.3 -> 95.0 mm
- net +15V: track 19.7 -> 29.3 mm
Other:
- board size 48.3 x 27.9 mm -> 53.3 x 27.9 mm
- board text added: "GND"
- board text added: "JLCJLCJLCJLC"
- board text added: "VIN"
- board text added: "VOUT"

Commit message: done : adjust back silkscreen
Other:
- board text added: "Up to 4A or 20W max WITHOUT WARRANTY of any kind !"
- board text removed: "15W should be OK 30W may be OK 45W is too much"
- board text removed: "WITHOUT WARRANTY of any kind !"
